File: KiCad_JLPCB_template_2layers/JLPCB_2layers.kicad_pcb (KiCad board)
At the start: 2 copper layers, 0 parts

Commit message: Starting up PCB
Parts:
- added C1: 10uF, Capacitor_SMD:CP_Elec_4x5.3, F.Cu at (135.8, 60.8)
- added C2: 0.22uF, Capacitor_SMD:C_1206_3216Metric_Pad1.33x1.80mm_HandSolder, F.Cu at (219.0, 96.0)
- added C3: 0.22uF, Capacitor_SMD:C_1206_3216Metric_Pad1.33x1.80mm_HandSolder, F.Cu at (236.0, 95.5)
- added C4: 100uF, Capacitor_SMD:CP_Elec_6.3x5.8, F.Cu at (139.3, 50.8)
- added C5: 0.22uF, Capacitor_SMD:C_1206_3216Metric_Pad1.33x1.80mm_HandSolder, F.Cu at (203.0, 96.0)
- added D11: 1N4148W, Diode_SMD:D_SOD-123, F.Cu at (219.0, 92.0)
- added D12: 1N4148W, Diode_SMD:D_SOD-123, F.Cu at (236.0, 92.0)
- added D13: 1N4148W, Diode_SMD:D_SOD-123, F.Cu at (203.0, 92.0)
- added GREEN: NSP_GRN, LED_THT:LED_D5.0mm, F.Cu at (234.0, 42.0)
- added GREEN: EWC_GRN, LED_THT:LED_D5.0mm, F.Cu at (159.2, 90.0)
- added GREEN: EWP_GRN, LED_THT:LED_D5.0mm, F.Cu at (130.7, 90.5)
- added GREEN: NSC_GRN, LED_THT:LED_D5.0mm, F.Cu at (201.2, 37.0)
- added H1: MountingHole, MountingHole:MountingHole_2.2mm_M2, F.Cu at (119.0, 26.0)
- added H2: MountingHole, MountingHole:MountingHole_2.2mm_M2, F.Cu at (247.0, 26.0)
- added H3: MountingHole, MountingHole:MountingHole_2.2mm_M2, F.Cu at (120.0, 117.0)
- added H4: MountingHole, MountingHole:MountingHole_2.2mm_M2, F.Cu at (247.0, 117.0)
- added J1: NS Connector, Connector_PinHeader_2.54mm:PinHeader_2x08_P2.54mm_Vertical, F.Cu at (154.4, 49.5)
- added J2: EW Connector, Connector_PinHeader_2.54mm:PinHeader_2x08_P2.54mm_Vertical, F.Cu at (154.4, 62.5)
- added J3: Control Logic Connector, Connector_PinHeader_2.54mm:PinHeader_2x05_P2.54mm_Vertical, F.Cu at (161.7, 37.0)
- added J4: +5V, my_footprints:Terminal_Block_5mm, F.Cu at (129.8, 38.8)
- added R1: 130R, Resistor_SMD:R_1206_3216Metric_Pad1.30x1.75mm_HandSolder, F.Cu at (219.5, 32.0)
- added R10: 130R, Resistor_SMD:R_1206_3216Metric_Pad1.30x1.75mm_HandSolder, F.Cu at (152.2, 82.7)
- added R11: 130R, Resistor_SMD:R_1206_3216Metric_Pad1.30x1.75mm_HandSolder, F.Cu at (147.5, 112.0)
- added R12: 130R, Resistor_SMD:R_1206_3216Metric_Pad1.30x1.75mm_HandSolder, F.Cu at (143.5, 112.0)
- added R13: 130R, Resistor_SMD:R_1206_3216Metric_Pad1.30x1.75mm_HandSolder, F.Cu at (139.5, 112.0)
- added R14: 130R, Resistor_SMD:R_1206_3216Metric_Pad1.30x1.75mm_HandSolder, F.Cu at (144.2, 82.7)
- added R15: 130R, Resistor_SMD:R_1206_3216Metric_Pad1.30x1.75mm_HandSolder, F.Cu at (140.2, 82.7)
- added R16: 130R, Resistor_SMD:R_1206_3216Metric_Pad1.30x1.75mm_HandSolder, F.Cu at (151.5, 112.0)
- added R17: 130R, Resistor_SMD:R_1206_3216Metric_Pad1.30x1.75mm_HandSolder, F.Cu at (192.0, 37.0)
- added R18: 130R, Resistor_SMD:R_1206_3216Metric_Pad1.30x1.75mm_HandSolder, F.Cu at (192.0, 47.0)
- added R19: 130R, Resistor_SMD:R_1206_3216Metric_Pad1.30x1.75mm_HandSolder, F.Cu at (192.0, 58.0)
- added R2: 130R, Resistor_SMD:R_1206_3216Metric_Pad1.30x1.75mm_HandSolder, F.Cu at (223.5, 32.0)
- added R20: 130R, Resistor_SMD:R_1206_3216Metric_Pad1.30x1.75mm_HandSolder, F.Cu at (169.5, 89.5)
- added R21: 130R, Resistor_SMD:R_1206_3216Metric_Pad1.30x1.75mm_HandSolder, F.Cu at (169.5, 100.0)
- added R22: 130R, Resistor_SMD:R_1206_3216Metric_Pad1.30x1.75mm_HandSolder, F.Cu at (169.5, 110.5)
- added R23: 130R, Resistor_SMD:R_1206_3216Metric_Pad1.30x1.75mm_HandSolder, F.Cu at (244.5, 42.0)
- added R24: 130R, Resistor_SMD:R_1206_3216Metric_Pad1.30x1.75mm_HandSolder, F.Cu at (244.5, 51.5)
- added R25: 130R, Resistor_SMD:R_1206_3216Metric_Pad1.30x1.75mm_HandSolder, F.Cu at (122.5, 90.5)
- added R26: 130R, Resistor_SMD:R_1206_3216Metric_Pad1.30x1.75mm_HandSolder, F.Cu at (122.5, 99.5)
- added R27: 47K, Resistor_SMD:R_1206_3216Metric_Pad1.30x1.75mm_HandSolder, F.Cu at (236.0, 84.0)
- added R28: 47K, Resistor_SMD:R_1206_3216Metric_Pad1.30x1.75mm_HandSolder, F.Cu at (219.0, 88.0)
- added R29: 47K, Resistor_SMD:R_1206_3216Metric_Pad1.30x1.75mm_HandSolder, F.Cu at (236.0, 88.0)
- added R3: 130R, Resistor_SMD:R_1206_3216Metric_Pad1.30x1.75mm_HandSolder, F.Cu at (220.0, 60.5)
- added R30: 47K, Resistor_SMD:R_1206_3216Metric_Pad1.30x1.75mm_HandSolder, F.Cu at (219.0, 84.0)
- added R31: 47K, Resistor_SMD:R_1206_3216Metric_Pad1.30x1.75mm_HandSolder, F.Cu at (203.0, 88.0)
- added R32: 47K, Resistor_SMD:R_1206_3216Metric_Pad1.30x1.75mm_HandSolder, F.Cu at (203.0, 84.0)
- added R4: 130R, Resistor_SMD:R_1206_3216Metric_Pad1.30x1.75mm_HandSolder, F.Cu at (216.0, 60.5)
- added R5: 130R, Resistor_SMD:R_1206_3216Metric_Pad1.30x1.75mm_HandSolder, F.Cu at (212.0, 60.5)
- added R6: 130R, Resistor_SMD:R_1206_3216Metric_Pad1.30x1.75mm_HandSolder, F.Cu at (215.5, 32.0)
- added R7: 130R, Resistor_SMD:R_1206_3216Metric_Pad1.30x1.75mm_HandSolder, F.Cu at (211.5, 32.0)
- added R8: 130R, Resistor_SMD:R_1206_3216Metric_Pad1.30x1.75mm_HandSolder, F.Cu at (224.0, 60.5)
- added R9: 130R, Resistor_SMD:R_1206_3216Metric_Pad1.30x1.75mm_HandSolder, F.Cu at (148.2, 82.7)
- added RED: EWP_RED, LED_THT:LED_D5.0mm, F.Cu at (130.7, 100.5)
- added RED: NSP_RED, LED_THT:LED_D5.0mm, F.Cu at (234.0, 51.5)
- added RED: NSC_RED, LED_THT:LED_D5.0mm, F.Cu at (201.2, 58.0)
- added RED: EWC_RED, LED_THT:LED_D5.0mm, F.Cu at (159.2, 110.5)
- added SW1: RST, my_footprints:tact_switch_5mm, F.Cu at (227.5, 91.5)
- added SW2: OVR, my_footprints:slide_switch_2.54mm, F.Cu at (196.0, 89.5)
- added SW3: EN, my_footprints:slide_switch_2.54mm, F.Cu at (211.5, 89.5)
- added U1: SM420561N, Display_7Segment:7SegmentLED_LTS6760_LTS6780, F.Cu at (212.9, 54.1)
- added U2: SM420561N, Display_7Segment:7SegmentLED_LTS6760_LTS6780, F.Cu at (140.9, 104.6)
- added U3: LM1117DT-3.3, Package_TO_SOT_SMD:SOT-223, F.Cu at (123.8, 56.8)
- added YELLOW: EWC_YLW, LED_THT:LED_D5.0mm, F.Cu at (159.2, 100.0)
- added YELLOW: NSC_YLW, LED_THT:LED_D5.0mm, F.Cu at (201.2, 47.5)
Routing:
- net /+5V: track 0.00 -> 15.8 mm
Other:
- board text added: "+"
- board text added: "+3V3"
- board text added: "+5V"
- board text added: "1"
- board text added: "2"
- board text added: "3"
- board text added: "A"
- board text added: "B"
- board text added: "C"
- board text added: "CAR"
- board text added: "Control Logic Connector"
- board text added: "D"
- board text added: "DP"
- board text added: "E"
- board text added: "E-W"
- board text added: "EAST-WEST TRAFFIC LIGHTS"
- board text added: "EN"
- board text added: "ENABLE"
- board text added: "EW Connector"
- board text added: "F"
- board text added: "G"
- board text added: "GND"
- board text added: "N-S"
- board text added: "NORTH-SOUTH TRAFFIC LIGHTS"
- board text added: "NS Connector"
- board text added: "OVERRIDE"
- board text added: "OVR"
- board text added: "PED"
- board text added: "R"
- board text added: "RESET"
- board text added: "RST"
- board text added: "Y"
